File: Open_ROV_Cape.sch (EAGLE design)
At the start: 19 parts, among them T1 2N2222, T2 TIP122

Commit message: started on new cape board
Parts:
- added JP4: (no value), microbuilder:HEADER-1X23
- added JP5, JP6, JP7: (no value), pinhead:PINHD-1X3
- added U$2: BEAGLEBONE_OUTLINE, microbuilder:BEAGLEBONE_OUTLINE
- added U$22, U$23: MOUNTINGHOLE3.0THIN, microbuilder:MOUNTINGHOLE3.0THIN
- JP1, JP2, JP3: device pinhead:PINHD-1X3 -> microbuilder:HEADER-1X23
Connections:
- new net 3.3V: JP3.22, JP4.2, U$2.VDD_3V3EXP@1, U$2.VDD_3V3EXP@2
- new net 5.0V: JP3.20, JP4.4, U$2.SYS_5V@1, U$2.SYS_5V@2
- new net AGND: JP2.19, U$2.UART5_RXD
- new net AVCC: JP1.4, U$2.GPIO2_12
- new net N$10: JP1.14, U$2.EHRPWM2A
- new net N$11: JP1.13, U$2.GPIO1_30
- new net N$12: JP1.12, U$2.GPIO1_4
- new net N$13: JP1.11, U$2.GPIO1_0
- new net N$14: JP1.10, U$2.GPIO2_22
- new net N$15: JP1.9, U$2.GPIO2_23
- new net N$16: JP1.8, U$2.UART5_CTSN
- new net N$21: JP1.3, U$2.GPIO2_10
- new net N$22: JP1.2, U$2.GPIO2_8
- new net N$23: JP1.1, U$2.GPIO2_6
- new net N$27: JP2.4, U$2.TIMER7
- new net N$28: JP2.5, U$2.TIMER6
- new net N$29: JP2.6, U$2.GPIO1_12
- new net N$30: JP2.7, U$2.GPIO0_26
- new net N$31: JP2.8, U$2.GPIO1_14
- new net N$32: JP2.9, U$2.GPIO2_1
- new net N$33: JP2.10, U$2.GPIO1_31
- new net N$34: JP2.11, U$2.GPIO1_5
- new net N$35: JP2.12, U$2.GPIO1_1
- new net N$36: JP2.13, U$2.GPIO1_29
- new net N$37: JP2.14, U$2.GPIO2_24
- new net N$38: JP2.15, U$2.GPIO2_25
- new net N$39: JP2.16, U$2.UART5_RTSN
- new net N$4: JP1.20, U$2.TIMER4
- new net N$40: JP2.17, U$2.UART3_RTSN
- new net N$41: JP2.18, U$2.UART3_CTSN
- new net N$43: JP2.20, U$2.GPIO2_13
- new net N$44: JP2.21, U$2.GPIO2_11
- new net N$45: JP2.22, U$2.GPIO2_9
- new net N$46: JP2.23, U$2.GPIO2_7
- new net N$47: JP1.22, U$2.GPIO1_6
- new net N$48: JP1.21, U$2.GPIO1_2
- new net N$49: JP3.21, U$2.VDD_5V@1
- new net N$5: JP1.19, U$2.TIMER5
- new net N$50: JP2.2, U$2.GPIO1_7
- new net N$51: JP3.19, U$2.PWR_BUT
- new net N$52: JP3.18, U$2.UART4_RXD
- new net N$53: JP3.17, U$2.UART4_TXD
- new net N$54: JP3.16, U$2.GPIO1_16
- new net N$55: JP3.15, U$2.I2C1_SCL
- new net N$56: JP3.14, U$2.I2C2_SCL
- new net N$57: JP3.13, U$2.UART2_TXD
- new net N$58: JP3.12, U$2.GPIO1_17
- new net N$59: JP3.11, U$2.GPIO3_21
- new net N$6: JP1.18, U$2.GPIO1_13
- new net N$60: JP3.10, U$2.GPIO3_19
- new net N$61: JP3.9, U$2.SPI1_DO
- new net N$62: JP3.8, U$2.SPI1_SCLK
- new net N$63: JP3.7, U$2.AIN4
- new net N$64: JP3.6, U$2.AIN6
- new net N$65: JP3.5, U$2.AIN2
- new net N$66: JP3.4, U$2.AIN0
- new net N$67: JP3.3, U$2.CLKOUT2
- new net N$68: JP2.3, U$2.GPIO1_3
- new net N$69: JP4.21, U$2.GPIO0_7
- new net N$7: JP1.17, U$2.EHRPWM2B
- new net N$72: JP4.3, U$2.VDD_5V@2
- new net N$74: JP4.5, U$2.SYS_RESETN
- new net N$75: JP4.6, U$2.GPIO1_28
- new net N$76: JP4.7, U$2.EHRPWM1A
- new net N$77: JP4.8, U$2.EHRPWM1B
- new net N$78: JP4.9, U$2.I2C1_SDA
- new net N$79: JP4.10, U$2.I2C2_SDA
- new net N$8: JP1.16, U$2.GPIO1_15
- new net N$80: JP4.11, U$2.UART2_RXD
- new net N$81: JP4.12, U$2.UART1_TXD
- new net N$82: JP4.13, U$2.UART1_RXD
- new net N$83: JP4.14, U$2.SPI1_CS0
- new net N$84: JP4.15, U$2.SPI1_DI
- new net N$85: JP4.16, U$2.VDD_ADC
- new net N$86: JP4.17, U$2.GNDA_ADC
- new net N$87: JP4.18, U$2.AIN5
- new net N$88: JP4.19, U$2.AIN3
- new net N$89: JP4.20, U$2.AIN1
- new net N$9: JP1.15, U$2.GPIO0_27
- new net N$92: JP5.1
- new net N$93: JP6.1
- new net N$94: JP7.1
- net GND: now also JP1.23, JP2.1, JP3.1, JP3.2, JP3.23, JP4.1, JP4.22, JP4.23, JP5.3, JP6.3, JP7.3, U$2.GND@1, U$2.GND@2, U$2.GND@3, U$2.GND@4, U$2.GND@5, U$2.GND@6, U$2.GND@7, U$2.GND@8; no longer JP1.3, JP2.3, JP3.3
- net N$17: now also JP1.7, U$2.UART4_RTSN; no longer JP1.1
- net N$18: now also JP1.6, U$2.UART4_CTSN; no longer JP2.1
- net N$19: now also JP1.5, U$2.UART5_TXD; no longer JP3.1
Other:
- moved on the sheet: C1, C2, C3, D1, D2, D3, IC1, IC2, Q1, R1, R2, R3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
